Commit message: Update main_revolute.urdf

File: urdf/main_revolute.urdf (robot description, URDF)
Before this commit: robot hand, 20 links, 19 joints
Joints:
- joint base_to_thumb_01: limit lower=-1.0 upper=1.0 effort=1000.0 velocity=0.5 -> lower=-2.0 upper=0.05 effort=1000.0 velocity=0.5
- joint thumb_01_to_02: limit lower=-1.0 upper=1.0 effort=1000.0 velocity=0.5 -> lower=-1.0 upper=0.05 effort=1000.0 velocity=0.5

Commit message: Update main_revolute.urdf

File: urdf/main_revolute.urdf (robot description, URDF)
Before this commit: robot hand, 20 links, 19 joints
Joints:
- joint base_to_thumb_01: axis 0 1 0 -> 1 1 0
